File: hardware/tent_map_amplitude.sch (KiCad schematic (older format))
At the start: 25 parts

Commit message: Use correct lm339AN part, auto-label components
Parts:
- removed U?: LM339, symbol Comparator:LM339
- added unit 2 of U1
- gave numbers to parts that had none: 22
Connections:
- net GND: now also U1.4
- net V+: now also U1.3 (VCC)
- net V-: now also U1.12 (GND)
- net at C1.1, R2.2, U2.5: now also U1.5
- net at R3.1: now also U1.2

Commit message: Assign temporary footprints, need to verify based on selection of components
Parts:
- C1, C2, C3, C4, C5, C6, C7: footprint (none) -> Capacitor_SMD:C_0805_2012Metric_Pad1.18x1.45mm_HandSolder
- R1, R2, R3, R4, R5, R6, R7, R8: footprint (none) -> Resistor_SMD:R_0805_2012Metric_Pad1.20x1.40mm_HandSolder
- RV1: footprint (none) -> Potentiometer_THT:Potentiometer_Bourns_3296Y_Vertical
Changed lines of the file:
@@
 F 0 "R6" H 6920 4296 50  0000 L CNN
 F 1 "1k" H 6920 4205 50  0000 L CNN
-F 2 "" V 6780 4250 50  0001 C CNN
+F 2 "Resistor_SMD:R_0805_2012Metric_Pad1.20x1.40mm_HandSolder" V 6780 4250 50  0001 C CNN
 F 3 "~" H 6850 4250 50  0001 C CNN
 	1    6850 4250
@@
 F 0 "R5" H 1930 3904 50  0000 R CNN
 F 1 "2k" H 1930 3995 50  0000 R CNN
-F 2 "" V 1930 3950 50  0001 C CNN
+F 2 "Resistor_SMD:R_0805_2012Metric_Pad1.20x1.40mm_HandSolder" V 1930 3950 50  0001 C CNN
 F 3 "~" H 2000 3950 50  0001 C CNN
 	1    2000 3950
@@
 F 0 "R4" V 1435 3600 50  0000 C CNN
 F 1 "220" V 1344 3600 50  0000 C CNN
-F 2 "" V 1480 3600 50  0001 C CNN
+F 2 "Resistor_SMD:R_0805_2012Metric_Pad1.20x1.40mm_HandSolder" V 1480 3600 50  0001 C CNN
 F 3 "~" H 1550 3600 50  0001 C CNN
 	1    1550 3600
@@
 F 0 "R2" V 1757 2200 50  0000 C CNN
 F 1 "220" V 1666 2200 50  0000 C CNN
-F 2 "" V 1480 2200 50  0001 C CNN
+F 2 "Resistor_SMD:R_0805_2012Metric_Pad1.20x1.40mm_HandSolder" V 1480 2200 50  0001 C CNN
 F 3 "~" H 1550 2200 50  0001 C CNN
 	1    1550 2200
@@
 F 0 "C1" H 3065 2546 50  0000 L CNN
 F 1 "1u" H 3065 2455 50  0000 L CNN
-F 2 "" H 2988 2350 50  0001 C CNN
+F 2 "Capacitor_SMD:C_0805_2012Metric_Pad1.18x1.45mm_HandSolder" H 2988 2350 50  0001 C CNN
 F 3 "~" H 2950 2500 50  0001 C CNN
 	1    2950 2500
@@
 F 0 "R3" V 5107 2300 50  0000 C CNN
 F 1 "10k" V 5016 2300 50  0000 C CNN
-F 2 "" V 4830 2300 50  0001 C CNN
+F 2 "Resistor_SMD:R_0805_2012Metric_Pad1.20x1.40mm_HandSolder" V 4830 2300 50  0001 C CNN
 F 3 "~" H 4900 2300 50  0001 C CNN
 	1    4900 2300
@@
 F 0 "R1" H 5370 1996 50  0000 L CNN
 F 1 "10k" H 5370 1905 50  0000 L CNN
-F 2 "" V 5230 1950 50  0001 C CNN
+F 2 "Resistor_SMD:R_0805_2012Metric_Pad1.20x1.40mm_HandSolder" V 5230 1950 50  0001 C CNN
 F 3 "~" H 5300 1950 50  0001 C CNN
 	1    5300 1950
@@
 F 0 "R7" H 9670 4446 50  0000 L CNN
 F 1 "1k" H 9670 4355 50  0000 L CNN
-F 2 "" V 9530 4400 50  0001 C CNN
+F 2 "Resistor_SMD:R_0805_2012Metric_Pad1.20x1.40mm_HandSolder" V 9530 4400 50  0001 C CNN
 F 3 "~" H 9600 4400 50  0001 C CNN
 	1    9600 4400
@@
 F 0 "R8" H 9670 4946 50  0000 L CNN
 F 1 "1k" H 9670 4855 50  0000 L CNN
-F 2 "" V 9530 4900 50  0001 C CNN
+F 2 "Resistor_SMD:R_0805_2012Metric_Pad1.20x1.40mm_HandSolder" V 9530 4900 50  0001 C CNN
 F 3 "~" H 9600 4900 50  0001 C CNN
 	1    9600 4900
@@
 F 0 "RV1" H 4030 4246 50  0000 R CNN
 F 1 "R_POT" H 4030 4155 50  0000 R CNN
-F 2 "" H 4100 4200 50  0001 C CNN
+F 2 "Potentiometer_THT:Potentiometer_Bourns_3296Y_Vertical" H 4100 4200 50  0001 C CNN
 F 3 "~" H 4100 4200 50  0001 C CNN
 	1    4100 4200
@@
 F 0 "C6" H 8415 5396 50  0000 L CNN
 F 1 "0.1u" H 8415 5305 50  0000 L CNN
-F 2 "" H 8338 5200 50  0001 C CNN
+F 2 "Capacitor_SMD:C_0805_2012Metric_Pad1.18x1.45mm_HandSolder" H 8338 5200 50  0001 C CNN
 F 3 "~" H 8300 5350 50  0001 C CNN
 	1    8300 5350
@@
 F 0 "C3" H 8465 4246 50  0000 L CNN
 F 1 "0.1u" H 8465 4155 50  0000 L CNN
-F 2 "" H 8388 4050 50  0001 C CNN
+F 2 "Capacitor_SMD:C_0805_2012Metric_Pad1.18x1.45mm_HandSolder" H 8388 4050 50  0001 C CNN
 F 3 "~" H 8350 4200 50  0001 C CNN
 	1    8350 4200
@@
 F 0 "C7" H 6315 6296 50  0000 L CNN
 F 1 "0.1u" H 6315 6205 50  0000 L CNN
-F 2 "" H 6238 6100 50  0001 C CNN
+F 2 "Capacitor_SMD:C_0805_2012Metric_Pad1.18x1.45mm_HandSolder" H 6238 6100 50  0001 C CNN
 F 3 "~" H 6200 6250 50  0001 C CNN
 	1    6200 6250
@@
 F 0 "C5" H 6615 5346 50  0000 L CNN
 F 1 "0.1u" H 6615 5255 50  0000 L CNN
-F 2 "" H 6538 5150 50  0001 C CNN
+F 2 "Capacitor_SMD:C_0805_2012Metric_Pad1.18x1.45mm_HandSolder" H 6538 5150 50  0001 C CNN
 F 3 "~" H 6500 5300 50  0001 C CNN
 	1    6500 5300
@@
 F 0 "C2" V 2798 4000 50  0000 C CNN
 F 1 "0.1u" V 2889 4000 50  0000 C CNN
-F 2 "" H 3088 3850 50  0001 C CNN
+F 2 "Capacitor_SMD:C_0805_2012Metric_Pad1.18x1.45mm_HandSolder" H 3088 3850 50  0001 C CNN
 F 3 "~" H 3050 4000 50  0001 C CNN
 	1    3050 4000
@@
 F 0 "C4" V 3050 4950 50  0000 C CNN
 F 1 "0.1u" V 3150 4950 50  0000 C CNN
-F 2 "" H 2938 4800 50  0001 C CNN
+F 2 "Capacitor_SMD:C_0805_2012Metric_Pad1.18x1.45mm_HandSolder" H 2938 4800 50  0001 C CNN
 F 3 "~" H 2900 4950 50  0001 C CNN
 	1    2900 4950

Commit message: Add test points, add WIP lf398 sample and hold circuit
Parts:
- removed J1: 22-23-2021, digikey-footprints:PinHeader_1x2_P2.54mm_Drill1.02mm, symbol dk_Rectangular-Connectors-Headers-Male-Pins:22-23-2021
- added C8, C9: 10u, Capacitor_THT:CP_Radial_D5.0mm_P2.00mm, symbol Device:CP1
- added C? (x4): 0.1u, Capacitor_SMD:C_0805_2012Metric_Pad1.18x1.45mm_HandSolder, symbol Device:C
- added TP1: Vc, TestPoint:TestPoint_Bridge_Pitch2.54mm_Drill1.0mm, symbol Connector:TestPoint
- added TP2: ana_out, TestPoint:TestPoint_Bridge_Pitch2.54mm_Drill1.0mm, symbol Connector:TestPoint
- added TP3: GND, TestPoint:TestPoint_Bridge_Pitch2.54mm_Drill1.0mm, symbol Connector:TestPoint
- added TP4: V+, TestPoint:TestPoint_Bridge_Pitch2.54mm_Drill1.0mm, symbol Connector:TestPoint
- added TP5: V-, TestPoint:TestPoint_Bridge_Pitch2.54mm_Drill1.0mm, symbol Connector:TestPoint
- added TP6: Vbuffer, TestPoint:TestPoint_Bridge_Pitch2.54mm_Drill1.0mm, symbol Connector:TestPoint
- added TP7, TP9: Vctrl, TestPoint:TestPoint_Bridge_Pitch2.54mm_Drill1.0mm, symbol Connector:TestPoint
- added TP8: ana_in, TestPoint:TestPoint_Bridge_Pitch2.54mm_Drill1.0mm, symbol Connector:TestPoint
- added U? (x4): LF398_DIP8, symbol Analog:LF398_DIP8
- RV1: footprint Potentiometer_THT:Potentiometer_Bourns_3296Y_Vertical -> Potentiometer_THT:Potentiometer_Bourns_3296W_Vertical
Connections:
- net GND: now also C8.2, C9.1, C?.2, C?.2, C?.2, C?.2, TP3.1, U?.7 (T), U?.7 (T), U?.7 (T), U?.7 (T)
- net V+: now also C8.1, TP4.1, U?.1 (V+), U?.1 (V+), U?.1 (V+), U?.1 (V+)
- net V-: now also C9.2, TP5.1, U?.4 (V-), U?.4 (V-), U?.4 (V-), U?.4 (V-)
- net at R6.2, U1.1, U3.3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: now also TP9.1
- net at U1.7: now also TP8.1
- net at C1.1, R2.2, U1.5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: now also TP1.1, U?.3 (I)
- net at R5.1, U2.1, U2.2: now also TP6.1
- net at RV1.2, U2.3: now also TP7.1
- net at R1.2, R3.2: now also TP2.1
- new net: C?.1, U?.6 (Ch) (x4)
- new net: U?.3 (I), U?.5 (x3)
Other:
- note added: "bypass caps for supply rails\nshould be tantalum or electrolytic"
- moved on the sheet: C1, C2, C3, C4, C5, C6, C7, D1, D2, R1, R2, R3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

Commit message: Complete PCB (unreviewed)
Parts:
- removed C?: 0.1u, Capacitor_SMD:C_0805_2012Metric_Pad1.18x1.45mm_HandSolder, symbol Device:C
- removed U?: LF398_DIP8, symbol Analog:LF398_DIP8
- added C10, C11, C12, C13, C14, C15: 0.1u, Capacitor_SMD:C_0805_2012Metric_Pad1.18x1.45mm_HandSolder, symbol Device:C
- added TP10: Vclock, TestPoint:TestPoint_Bridge_Pitch2.54mm_Drill1.0mm, symbol Connector:TestPoint
- added TP11: Vsn+1, TestPoint:TestPoint_Bridge_Pitch2.54mm_Drill1.0mm, symbol Connector:TestPoint
- added TP12: Vclock-, TestPoint:TestPoint_Bridge_Pitch2.54mm_Drill1.0mm, symbol Connector:TestPoint
- added TP13: Vsn+1/2, TestPoint:TestPoint_Bridge_Pitch2.54mm_Drill1.0mm, symbol Connector:TestPoint
- added TP14: Vsn, TestPoint:TestPoint_Bridge_Pitch2.54mm_Drill1.0mm, symbol Connector:TestPoint
- C16, C17, C18: renamed from C?; footprint Capacitor_SMD:C_0805_2012Metric_Pad1.18x1.45mm_HandSolder -> Capacitor_THT:C_Rect_L10.3mm_W5.0mm_P7.50mm_MKS4
- U4, U5, U6: renamed from U?; footprint (none) -> digikey-footprints:DIP-8_W7.62mm
Connections:
- net GND: now also C10.1, C11.1, C12.1, C13.1, C14.1, C15.1
- net V+: now also C10.2, C12.2, C14.2
- net V-: now also C11.2, C13.2, C15.2
- net at U4.5, U5.3 (I): now also TP11.1
- net at U5.5, U6.3 (I): now also TP13.1
- net at U5.8 (Hold): now also TP12.1
- net at U4.8 (Hold): now also U6.8 (Hold), TP10.1
- net at U6.5: now also TP14.1
Other:
- note added: "decoupling caps for lf398s\n"
- note added: "need a clock double the speed of the regular clock for sampling\nfirst and third lf398's need to sample at positive going edge of the double clock\nand 2nd lf398 needs to sample at negative going edge of the double clock"
- note added: "sampling circuit relies on fpga/digital\n logic to give proper sampling pulses based \non main clock"
- note added: "sampling should use polypropolene caps as they have less hysterisis than other cap types\n"
- moved on the sheet: C1, C16, C17, C18, C2, C4, C8, C9, R1, R2, R3, R4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

Commit message: update pcb and schematic to have 3.3V input for interfacing with DE-10 nano
Parts:
- added TP15: V+3.3, TestPoint:TestPoint_Bridge_Pitch2.54mm_Drill1.0mm, symbol Connector:TestPoint
- R1, R3: value 10k -> 1k
- TP9: value Vctrl -> VcompA
Connections:
- net V+: no longer R1.1
- net at TP6.1, U2.1, U2.2: now also R5.2; no longer R5.1
- net at R4.2, U2.6: now also R5.1; no longer R5.2
- new net +3V3: R1.1, TP15.1
Changed lines of the file:
@@
 Wire Wire Line
 	1850 6500 1850 6000
-$Comp
-L Device:R R5
-U 1 1 5F95B93C
-P 1850 5650
-F 0 "R5" H 1780 5604 50  0000 R CNN
-F 1 "2k" H 1780 5695 50  0000 R CNN
-F 2 "Resistor_SMD:R_0805_2012Metric_Pad1.20x1.40mm_HandSolder" V 1780 5650 50  0001 C CNN
-F 3 "~" H 1850 5650 50  0001 C CNN
-	1    1850 5650
-	-1   0    0    1
-$EndComp
-Wire Wire Line
-	1850 6000 1850 5800
 Connection ~ 1850 6000
 $Comp
@@
 $EndComp
 Wire Wire Line
-	1850 5500 1850 5300
-Wire Wire Line
 	1550 5300 1850 5300
 Wire Wire Line
@@
 Wire Wire Line
 	1850 4800 1850 5300
-Connection ~ 1850 5300
 Wire Wire Line
 	1250 5300 850  5300
@@
 P 4750 4000
 F 0 "R3" V 4957 4000 50  0000 C CNN
-F 1 "10k" V 4866 4000 50  0000 C CNN
+F 1 "1k" V 4866 4000 50  0000 C CNN
 F 2 "Resistor_SMD:R_0805_2012Metric_Pad1.20x1.40mm_HandSolder" V 4680 4000 50  0001 C CNN
 F 3 "~" H 4750 4000 50  0001 C CNN
@@
 P 5150 3650
 F 0 "R1" H 5220 3696 50  0000 L CNN
-F 1 "10k" H 5220 3605 50  0000 L CNN
+F 1 "1k" H 5220 3605 50  0000 L CNN
 F 2 "Resistor_SMD:R_0805_2012Metric_Pad1.20x1.40mm_HandSolder" V 5080 3650 50  0001 C CNN
 F 3 "~" H 5150 3650 50  0001 C CNN
@@
 Wire Wire Line
 	4600 4000 4200 4000
-$Comp
-L power:V+ #PWR01
-U 1 1 5F98106D
-P 5150 3450
-F 0 "#PWR01" H 5150 3300 50  0001 C CNN
-F 1 "V+" H 5165 3623 50  0000 C CNN
-F 2 "" H 5150 3450 50  0001 C CNN
-F 3 "" H 5150 3450 50  0001 C CNN
-	1    5150 3450
-	1    0    0    -1
-$EndComp
 Wire Wire Line
 	5150 3450 5150 3500
@@
 $EndComp
 $Comp
-L power:V+ #PWR04
-U 1 1 5F91EF5C
-P 3900 4350
-F 0 "#PWR04" H 3900 4200 50  0001 C CNN
-F 1 "V+" H 3915 4523 50  0000 C CNN
-F 2 "" H 3900 4350 50  0001 C CNN
-F 3 "" H 3900 4350 50  0001 C CNN
-	1    3900 4350
-	-1   0    0    1
-$EndComp
-Wire Wire Line
-	3900 4350 3900 4200
-$Comp
-L power:V- #PWR02
-U 1 1 5F9237E3
-P 3900 3650
-F 0 "#PWR02" H 3900 3525 50  0001 C CNN
-F 1 "V-" H 3915 3823 50  0000 C CNN
-F 2 "" H 3900 3650 50  0001 C CNN
-F 3 "" H 3900 3650 50  0001 C CNN
-	1    3900 3650
-	1    0    0    -1
-$EndComp
-Wire Wire Line
-	3900 3650 3900 3800
-$Comp
 L Connector:TestPoint TP2
 U 1 1 5F93CE4E
@@
 P 7100 5650
 F 0 "TP9" H 7042 5676 50  0000 R CNN
-F 1 "Vctrl" H 7042 5767 50  0000 R CNN
+F 1 "VcompA" H 7042 5767 50  0000 R CNN
 F 2 "TestPoint:TestPoint_Bridge_Pitch2.54mm_Drill1.0mm" H 7300 5650 50  0001 C CNN
 F 3 "~" H 7300 5650 50  0001 C CNN
@@
 Wire Wire Line
 	4750 1950 4750 1400
+Wire Wire Line
+	3900 3600 3900 3800
+$Comp
+L power:+3.3V #PWR0125
+U 1 1 5F960506
+P 5150 3450
+F 0 "#PWR0125" H 5150 3300 50  0001 C CNN
+F 1 "+3.3V" H 5165 3623 50  0000 C CNN
+F 2 "" H 5150 3450 50  0001 C CNN
+F 3 "" H 5150 3450 50  0001 C CNN
+	1    5150 3450
+	1    0    0    -1
+$EndComp
+$Comp
+L power:V+ #PWR0126
+U 1 1 5F9610DD
+P 3900 4350
+F 0 "#PWR0126" H 3900 4200 50  0001 C CNN
+F 1 "V+" H 3915 4523 50  0000 C CNN
+F 2 "" H 3900 4350 50  0001 C CNN
+F 3 "" H 3900 4350 50  0001 C CNN
+	1    3900 4350
+	-1   0    0    1
+$EndComp
+Wire Wire Line
+	3900 4200 3900 4350
+$Comp
+L power:V- #PWR0127
+U 1 1 5F96862B
+P 3900 3600
+F 0 "#PWR0127" H 3900 3475 50  0001 C CNN
+F 1 "V-" H 3915 3773 50  0000 C CNN
+F 2 "" H 3900 3600 50  0001 C CNN
+F 3 "" H 3900 3600 50  0001 C CNN
+	1    3900 3600
+	1    0    0    -1
+$EndComp
+$Comp
+L Device:R R5
+U 1 1 5F97CAAC
+P 1850 5550
+F 0 "R5" V 1735 5550 50  0000 C CNN
+F 1 "2k" V 1644 5550 50  0000 C CNN
+F 2 "Resistor_SMD:R_0805_2012Metric_Pad1.20x1.40mm_HandSolder" V 1780 5550 50  0001 C CNN
+F 3 "~" H 1850 5550 50  0001 C CNN
+	1    1850 5550
+	1    0    0    -1
+$EndComp
+Wire Wire Line
+	1850 5400 1850 5300
+Connection ~ 1850 5300
+Wire Wire Line
+	1850 5700 1850 6000
+$Comp
+L Connector:TestPoint TP15
+U 1 1 5F9C9A10
+P 5650 3400
+F 0 "TP15" V 5550 3450 50  0000 C CNN
+F 1 "V+3.3" V 5450 3450 50  0000 C CNN
+F 2 "TestPoint:TestPoint_Bridge_Pitch2.54mm_Drill1.0mm" H 5850 3400 50  0001 C CNN
+F 3 "~" H 5850 3400 50  0001 C CNN
+	1    5650 3400
+	1    0    0    -1
+$EndComp
+Wire Wire Line
+	5650 3400 5650 3500
+Wire Wire Line
+	5650 3500 5150 3500
+Connection ~ 5150 3500
 $EndSCHEMATC

Commit message: use 3.3v for logic level for input comparator
Connections:
- net +3V3: now also R7.1
- net V+: no longer R7.1
Changed lines of the file:
@@
 Wire Wire Line
 	9450 5750 9450 5900
-$Comp
-L power:V+ #PWR013
-U 1 1 5F9A83F7
-P 9450 4750
-F 0 "#PWR013" H 9450 4600 50  0001 C CNN
-F 1 "V+" H 9465 4923 50  0000 C CNN
-F 2 "" H 9450 4750 50  0001 C CNN
-F 3 "" H 9450 4750 50  0001 C CNN
-	1    9450 4750
-	1    0    0    -1
-$EndComp
 Wire Wire Line
 	9450 4750 9450 4950
@@
 	5650 3500 5150 3500
 Connection ~ 5150 3500
+$Comp
+L power:+3.3V #PWR?
+U 1 1 5F966AFF
+P 9450 4750
+F 0 "#PWR?" H 9450 4600 50  0001 C CNN
+F 1 "+3.3V" H 9465 4923 50  0000 C CNN
+F 2 "" H 9450 4750 50  0001 C CNN
+F 3 "" H 9450 4750 50  0001 C CNN
+	1    9450 4750
+	1    0    0    -1
+$EndComp
 $EndSCHEMATC

Commit message: Add variable resistor 2
Parts:
- removed R5: 2k, Resistor_SMD:R_0805_2012Metric_Pad1.20x1.40mm_HandSolder, symbol Device:R
- added C? (x2): dnc, Capacitor_THT:C_Rect_L10.3mm_W5.0mm_P7.50mm_MKS4, symbol Device:C
- added RV2: R_POT, Potentiometer_THT:Potentiometer_Bourns_3296W_Vertical, symbol Device:R_POT
- R1, R3, R6, R7, R8: value 1k -> 10k
Connections:
- net GND: now also C?.2
- net at TP6.1, U2.1, U2.2: now also RV2.2, RV2.3
- net at R4.2, U2.6: now also RV2.1
- net at C16.1, U4.6 (Ch): now also C?.1
Other:
- moved on the sheet: TP11
Changed lines of the file:
@@
 P 6700 4950
 F 0 "R6" H 6770 4996 50  0000 L CNN
-F 1 "1k" H 6770 4905 50  0000 L CNN
+F 1 "10k" H 6770 4905 50  0000 L CNN
 F 2 "Resistor_SMD:R_0805_2012Metric_Pad1.20x1.40mm_HandSolder" V 6630 4950 50  0001 C CNN
 F 3 "~" H 6700 4950 50  0001 C CNN
@@
 P 4750 4000
 F 0 "R3" V 4957 4000 50  0000 C CNN
-F 1 "1k" V 4866 4000 50  0000 C CNN
+F 1 "10k" V 4866 4000 50  0000 C CNN
 F 2 "Resistor_SMD:R_0805_2012Metric_Pad1.20x1.40mm_HandSolder" V 4680 4000 50  0001 C CNN
 F 3 "~" H 4750 4000 50  0001 C CNN
@@
 P 5150 3650
 F 0 "R1" H 5220 3696 50  0000 L CNN
-F 1 "1k" H 5220 3605 50  0000 L CNN
+F 1 "10k" H 5220 3605 50  0000 L CNN
 F 2 "Resistor_SMD:R_0805_2012Metric_Pad1.20x1.40mm_HandSolder" V 5080 3650 50  0001 C CNN
 F 3 "~" H 5150 3650 50  0001 C CNN
@@
 P 9450 5100
 F 0 "R7" H 9520 5146 50  0000 L CNN
-F 1 "1k" H 9520 5055 50  0000 L CNN
+F 1 "10k" H 9520 5055 50  0000 L CNN
 F 2 "Resistor_SMD:R_0805_2012Metric_Pad1.20x1.40mm_HandSolder" V 9380 5100 50  0001 C CNN
 F 3 "~" H 9450 5100 50  0001 C CNN
@@
 P 9450 5600
 F 0 "R8" H 9520 5646 50  0000 L CNN
-F 1 "1k" H 9520 5555 50  0000 L CNN
+F 1 "10k" H 9520 5555 50  0000 L CNN
 F 2 "Resistor_SMD:R_0805_2012Metric_Pad1.20x1.40mm_HandSolder" V 9380 5600 50  0001 C CNN
 F 3 "~" H 9450 5600 50  0001 C CNN
@@
 $EndComp
 Wire Wire Line
-	3300 2200 3300 1950
+	3300 2000 3300 1950
 Connection ~ 3300 1950
 $Comp
 L Connector:TestPoint TP11
 U 1 1 5F931721
-P 3300 2200
-F 0 "TP11" V 3254 2388 50  0000 L CNN
-F 1 "Vsn+1" V 3345 2388 50  0000 L CNN
-F 2 "TestPoint:TestPoint_Bridge_Pitch2.54mm_Drill1.0mm" H 3500 2200 50  0001 C CNN
-F 3 "~" H 3500 2200 50  0001 C CNN
-	1    3300 2200
+P 3300 2000
+F 0 "TP11" V 3254 2188 50  0000 L CNN
+F 1 "Vsn+1" V 3345 2188 50  0000 L CNN
+F 2 "TestPoint:TestPoint_Bridge_Pitch2.54mm_Drill1.0mm" H 3500 2000 50  0001 C CNN
+F 3 "~" H 3500 2000 50  0001 C CNN
+	1    3300 2000
 	-1   0    0    1
 $EndComp
@@
 U 1 1 5FB8D6B7
 P 4000 2500
-F 0 "C17" H 4115 2546 50  0000 L CNN
-F 1 "0.1u" H 4115 2455 50  0000 L CNN
+F 0 "C17" H 3700 2450 50  0000 L CNN
+F 1 "0.1u" H 3700 2350 50  0000 L CNN
 F 2 "Capacitor_THT:C_Rect_L10.3mm_W5.0mm_P7.50mm_MKS4" H 4038 2350 50  0001 C CNN
 F 3 "~" H 4000 2500 50  0001 C CNN
@@
 U 1 1 5FB6213D
 P 2850 2500
-F 0 "C16" H 2965 2546 50  0000 L CNN
-F 1 "0.1u" H 2965 2455 50  0000 L CNN
+F 0 "C16" H 2600 2500 50  0000 L CNN
+F 1 "0.1u" H 2600 2400 50  0000 L CNN
 F 2 "Capacitor_THT:C_Rect_L10.3mm_W5.0mm_P7.50mm_MKS4" H 2888 2350 50  0001 C CNN
 F 3 "~" H 2850 2500 50  0001 C CNN
@@
 	1    0    0    -1
 $EndComp
-$Comp
-L Device:R R5
-U 1 1 5F97CAAC
-P 1850 5550
-F 0 "R5" V 1735 5550 50  0000 C CNN
-F 1 "2k" V 1644 5550 50  0000 C CNN
-F 2 "Resistor_SMD:R_0805_2012Metric_Pad1.20x1.40mm_HandSolder" V 1780 5550 50  0001 C CNN
-F 3 "~" H 1850 5550 50  0001 C CNN
-	1    1850 5550
-	1    0    0    -1
-$EndComp
 Wire Wire Line
 	1850 5400 1850 5300
 Connection ~ 1850 5300
 Wire Wire Line
-	1850 5700 1850 6000
+	1850 5700 1850 5800
 $Comp
 L Connector:TestPoint TP15
@@
 Connection ~ 5150 3500
 $Comp
-L power:+3.3V #PWR?
+L power:+3.3V #PWR0128
 U 1 1 5F966AFF
 P 9450 4750
-F 0 "#PWR?" H 9450 4600 50  0001 C CNN
+F 0 "#PWR0128" H 9450 4600 50  0001 C CNN
 F 1 "+3.3V" H 9465 4923 50  0000 C CNN
 F 2 "" H 9450 4750 50  0001 C CNN
@@
 	1    0    0    -1
 $EndComp
+$Comp
+L Device:R_POT RV2
+U 1 1 5F97AD16
+P 1850 5550
+F 0 "RV2" H 1780 5596 50  0000 R CNN
+F 1 "R_POT" H 1780 5505 50  0000 R CNN
+F 2 "Potentiometer_THT:Potentiometer_Bourns_3296W_Vertical" H 1850 5550 50  0001 C CNN
+F 3 "~" H 1850 5550 50  0001 C CNN
+	1    1850 5550
+	-1   0    0    -1
+$EndComp
+Wire Wire Line
+	1700 5550 1600 5550
+Wire Wire Line
+	1600 5550 1600 5800
+Wire Wire Line
+	1600 5800 1850 5800
+Connection ~ 1850 5800
+Wire Wire Line
+	1850 5800 1850 6000
+$Comp
+L Device:C C?
+U 1 1 5F984C5C
+P 3100 2500
+F 0 "C?" H 3150 2350 50  0000 L CNN
+F 1 "dnc" H 3215 2455 50  0000 L CNN
+F 2 "Capacitor_THT:C_Rect_L10.3mm_W5.0mm_P7.50mm_MKS4" H 3138 2350 50  0001 C CNN
+F 3 "~" H 3100 2500 50  0001 C CNN
+	1    3100 2500
+	1    0    0    -1
+$EndComp
+Wire Wire Line
+	3100 2350 2850 2350
+Connection ~ 2850 2350
+Wire Wire Line
+	3100 2650 2850 2650
+Connection ~ 2850 2650
+$Comp
+L Device:C C?
+U 1 1 5F99B1C9
+P 4200 2550
+F 0 "C?" H 4250 2400 50  0000 L CNN
+F 1 "dnc" H 4315 2505 50  0000 L CNN
+F 2 "Capacitor_THT:C_Rect_L10.3mm_W5.0mm_P7.50mm_MKS4" H 4238 2400 50  0001 C CNN
+F 3 "~" H 4200 2550 50  0001 C CNN
+	1    4200 2550
+	1    0    0    -1
+$EndComp
